Commit message: Update RViz configuration and URDF properties for improved robot representation

File: ros2_control_diffbot_description/diffbot/urdf/diffbot_description.urdf.xacro (robot description, xacro)
@@ -5,13 +5,13 @@
   <xacro:property name="PI" value="3.1415926535897931"/>
   <xacro:property name="base_mass" value="0.3" /> <!-- arbitrary value for base mass -->
-  <xacro:property name="base_width" value="0.1" />
-  <xacro:property name="base_length" value="0.1" />
-  <xacro:property name="base_height" value="0.05" />
+  <xacro:property name="base_width" value="0.16" />
+  <xacro:property name="base_length" value="0.115" />
+  <xacro:property name="base_height" value="0.049" />
   <xacro:property name="wheel_mass" value="0.3" /> <!-- arbitrary value for wheel mass -->
-  <xacro:property name="wheel_len" value="0.020" />
-  <xacro:property name="wheel_radius" value="0.015" />
+  <xacro:property name="wheel_len" value="0.018" />
+  <xacro:property name="wheel_radius" value="0.021" />
   <xacro:property name="caster_wheel_mass" value="0.1" /> <!-- arbitrary value for caster wheel mass -->
-  <xacro:property name="caster_wheel_radius" value="0.015" />
-  <xacro:property name="z_offset" value="-${base_height/2}" /> <!-- Space btw top of beam and the each joint -->
+  <xacro:property name="caster_wheel_radius" value="0.021" />
+  <xacro:property name="z_offset" value="-${base_height/2 - 0.01}" /> <!-- Space btw top of beam and the each joint -->
   <!-- Base Link -->
   <link name="${prefix}base_link">
@@ -27,5 +27,5 @@
         <box size="${base_width} ${base_length} ${base_height}"/>
       </geometry>
-      <material name="orange"/>
+      <material name="white"/>
     </visual>
     <inertial>
@@ -41,5 +41,5 @@
       <parent link="${prefix}base_link"/>
       <child link="${prefix}left_wheel"/>
-      <origin xyz="0 -${base_width/2} ${z_offset}" rpy="0 0 0"/>
+      <origin xyz="0.04 -${base_width/2} ${z_offset}" rpy="0 0 0"/>
       <axis xyz="0 1 0"/>
       <dynamics damping="0.2"/>
@@ -73,5 +73,5 @@
       <parent link="${prefix}base_link"/>
       <child link="${prefix}right_wheel"/>
-      <origin xyz="0 ${base_width/2} ${z_offset}" rpy="0 0 0"/>
+      <origin xyz="0.04 ${base_width/2} ${z_offset}" rpy="0 0 0"/>
       <axis xyz="0 1 0"/>
       <dynamics damping="0.2"/>
@@ -100,33 +100,4 @@
           iyy="${wheel_mass / 12.0 * (3*wheel_radius*wheel_radius + wheel_len*wheel_len)}" iyz="0.0"
           izz="${wheel_mass / 2.0 * wheel_radius*wheel_radius}"/>
-        </inertial>
-      </link>
-    <joint name="${prefix}caster_frontal_wheel_joint" type="fixed">
-      <parent link="${prefix}base_link"/>
-      <child link="${prefix}caster_frontal_wheel"/>
-      <origin xyz="${base_width/2 - caster_wheel_radius} 0 ${z_offset}" rpy="0 0 0"/>
-    </joint>
-    <!-- caster frontal wheel Link -->
-    <link name="${prefix}caster_frontal_wheel">
-      <collision>
-        <origin xyz="0 0 0" rpy="0 0 0"/>
-        <geometry>
-          <sphere radius="${caster_wheel_radius}"/>
-        </geometry>
-      </collision>
-      <visual>
-        <origin xyz="0 0 0" rpy="0 0 0"/>
-        <geometry>
-          <sphere radius="${caster_wheel_radius}"/>
-        </geometry>
-        <material name="white"/>
-      </visual>
-      <inertial>
-        <origin xyz="0 0 0" rpy="0 0 0"/>
-        <mass value="${caster_wheel_mass}"/>
-        <inertia
-          ixx="${caster_wheel_mass * 0.4 * (caster_wheel_radius * caster_wheel_radius)}" ixy="0.0" ixz="0.0"
-          iyy="${caster_wheel_mass * 0.4 * (caster_wheel_radius * caster_wheel_radius)}" iyz="0.0"
-          izz="${caster_wheel_mass * 0.4 * (caster_wheel_radius * caster_wheel_radius)}"/>
         </inertial>
       </link>

Commit message: Update VSCode settings and modify URDF properties for caster wheel radius and material color

File: ros2_control_diffbot_description/diffbot/urdf/diffbot_description.urdf.xacro (robot description, xacro)
@@ -12,5 +12,5 @@
   <xacro:property name="wheel_radius" value="0.021" />
   <xacro:property name="caster_wheel_mass" value="0.1" /> <!-- arbitrary value for caster wheel mass -->
-  <xacro:property name="caster_wheel_radius" value="0.021" />
+  <xacro:property name="caster_wheel_radius" value="${0.018}" />
   <xacro:property name="z_offset" value="-${base_height/2 - 0.01}" /> <!-- Space btw top of beam and the each joint -->
   <!-- Base Link -->
@@ -59,5 +59,5 @@
           <cylinder length="${wheel_len}" radius="${wheel_radius}"/>
         </geometry>
-        <material name="black"/>
+        <material name="grey"/>
       </visual>
       <inertial>
@@ -91,5 +91,5 @@
           <cylinder length="${wheel_len}" radius="${wheel_radius}"/>
         </geometry>
-        <material name="black"/>
+        <material name="grey"/>
       </visual>
       <inertial>
